File: Pure ADSR.brd (EAGLE design)
At the start: 33.6 x 100 mm, 44 parts, among them Q1 20MHz, U1 ATMEGA328P

Commit message: ADSR 2.1
Parts:
- removed BUT: (no value), INSTRUO:PB6149L
- removed IN, OUT: (no value), INSTRUO:S_JACK
- removed JP1: M05X2SHD, SparkFun-Connectors:2X5-SHROUDED
- removed MODE: (no value), INSTRUO:TOGGLE_ON_OFF_ON
- removed POT_A, POT_D, POT_R, POT_S: (no value), INSTRUO:Q-POT
- removed U$3: DUAL_OPAMP, INSTRUO:DUAL_OPAMP
- removed U$4: 7805, INSTRUO:V-REG
- removed U$5: (no value), INSTRUO_logos:SIG_LARGE_STOP
- removed U$6: (no value), INSTRUO_logos:SIG_LARGE_COPPER
- removed U1: ATMEGA328P, SparkFun-DigitalIC:TQFP32-08
- added ATTACK, DECAY, RELEASE, SUSTAIN: 100k, GMSN:POTENTIOMETER_9MM
- added IC1: 78M05, GMSN:TO252
- added IC2: OPAMP_DUALD, GMSN:SO08
- added IC3: MCP4921, GMSN:SOIC8
- added IC4: ATMEGA328P, GMSN:TQFP32-08
- added MODESW: ON_OFF_ON, GMSN:TOGGLE_ON_OFF_ON
- added OUTPUT, TRIGATEIN: SOCKET_MONO_3.5MMPJ301M-12, GMSN:PJ301M-12
- added POWER: HEADER2X5SHD, GMSN:2X5-SHROUDED
- added T1: MMBT2222A, GMSN:SOT23
- added TRIGGER: PB6149L-5, GMSN:PB6149L
- C1, C2, C6: device rcl:C0805K -> GMSN:C0805
- C10, C11, C12, C8, C9: value 0.1u -> 100nF; device rcl:C0805K -> GMSN:C0805
- C3: value 560p -> 10nF; device rcl:C0805K -> GMSN:C0805
- C4, C5, C7: device rcl:153CLV-0505 -> GMSN:153CLV-0505
- D1, D2: value (none) -> STTH102A; device adafruit:SMADIODE -> GMSN:SMADIODE
- ISP1: value AVRISP-6 -> HEADER2X3-6; device adafruit:AVRISP -> GMSN:AVRISP
- Q1: device adafruit:HC49UP -> GMSN:HC49UP
- R1: value 47K -> 56k; device rcl:R0805 -> GMSN:R0805
- R10, R8: value 1K -> 1k; device rcl:R0805 -> GMSN:R0805
- R11, R12, R6: value 100K -> 100k; device rcl:R0805 -> GMSN:R0805
- R2: value 30K -> 30k; device rcl:R0805 -> GMSN:R0805
- R3: value 50K -> 56k; device rcl:R0805 -> GMSN:R0805
- R4, R7: device rcl:R0805 -> GMSN:R0805
- R5, R9: value 10K -> 10k; device rcl:R0805 -> GMSN:R0805
- U$1: value 2N3904 -> (none); device INSTRUO:TRANSISTOR_SINGLE_N-TYPE -> gmsnLogo:GMSN!_LOGO
- U$2: value MCP4921 -> (none); device INSTRUO:SOIC8 -> gmsnLogo:GMSN!_LOGO
- moved U$1 72.8 mm to (17.5, 19.1), turned to 0 degrees
- moved U$2 41.6 mm to (18.3, 44.5), flipped to the top, turned to 0 degrees
- moved R5 29.8 mm to (2.86, 86.0), flipped to the top
- moved R10 27.0 mm to (4.29, 80.2), flipped to the top
- moved R6 27.0 mm to (4.29, 98.9), flipped to the top
- moved R7 27.0 mm to (4.29, 94.0), flipped to the top
- moved Q1 26.7 mm to (4.45, 108.6), flipped to the top
- moved R11 23.5 mm to (6.03, 84.9), flipped to the top
- moved R12 23.5 mm to (6.03, 74.6), flipped to the top
- moved C12 23.2 mm to (29.4, 113.8), flipped to the top
- moved R9 22.5 mm to (6.51, 65.6), flipped to the top
- moved C4 21.6 mm to (6.99, 24.8), flipped to the top
- moved C5 21.6 mm to (28.6, 24.8), flipped to the top
- moved D1 21.6 mm to (6.99, 19.1), flipped to the top
- moved D2 20.3 mm to (27.9, 19.1), flipped to the top
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Connections:
- new net 5V: ATTACK.P$3, C10.1, C11.1, C12.1, DECAY.P$3, IC3.1, IC3.6, IC4.18, IC4.4, IC4.6, ISP1.2, R10.2, R5.2, R9.2, RELEASE.P$3, SUSTAIN.P$3
- net +12V: now also IC1.1, IC2.8; no longer U$3.+VCC, U$4.1
- net +5V: now also IC1.2; no longer C10.1, C11.1, C12.1, ISP1.2, POT_A.P$3, POT_D.P$3, POT_R.P$3, POT_S.P$3, R10.2, R5.2, R9.2, U$2.1, U$2.6, U$4.3, U1.18, U1.4, U1.6
- net -12V: now also IC2.4; no longer U$3.-VCC
- net B_TRIG: now also IC4.1, IC4.2, TRIGGER.1, TRIGGER.2; no longer BUT.1, BUT.3, U1.1, U1.2
- net CS: now also IC3.2, IC4.14; no longer U$2.2, U1.14
- net GND: now also ATTACK.P$1, DECAY.P$1, IC1.3, IC3.5, IC3.7, IC4.21, IC4.3, IC4.5, OUTPUT.GND, POWER.3, POWER.4, POWER.5, POWER.6, POWER.7, POWER.8, RELEASE.P$1, SUSTAIN.P$1, T1.2, TRIGATEIN.GND, TRIGGER.3, TRIGGER.4; no longer BUT.2, BUT.4, IN.GND, JP1.3, JP1.4, JP1.5, JP1.6, JP1.7, JP1.8, OUT.GND, POT_A.P$1, POT_D.P$1, POT_R.P$1, POT_S.P$1, U$1.E, U$2.5, U$2.7, U$4.4, U1.21, U1.3, U1.5
- net MISO: now also IC4.16; no longer U1.16
- net MOSI: now also IC3.4, IC4.15; no longer U$2.4, U1.15
- net N$1: now also IC4.7; no longer U1.7
- net N$10: now also POWER.1, POWER.2; no longer JP1.1, JP1.2
- net N$11: now also IC2.1; no longer U$3.1OUT
- net N$12: now also MODESW.2; no longer MODE.2
- net N$15: now also T1.1; no longer U$1.B
- net N$18: now also TRIGATEIN.TIP; no longer IN.TIP
- net N$2: now also IC4.8; no longer U1.8
- net N$3: now also IC3.8; no longer U$2.8
- net N$4: now also IC2.3, IC2.5; no longer U$3.+1IN, U$3.+2IN
- net N$5: now also IC2.2; no longer U$3.-1IN
- net N$6: now also OUTPUT.TIP; no longer OUT.TIP
- net N$7: now also IC2.6, IC2.7, TRIGGER.A; no longer BUT.A, U$3.-2IN, U$3.2OUT
- net N$8: now also TRIGGER.K; no longer BUT.K
- net N$9: now also POWER.10, POWER.9; no longer JP1.10, JP1.9
- net POT_A: now also ATTACK.P$2, IC4.26; no longer POT_A.P$2, U1.26
- net POT_D: now also DECAY.P$2, IC4.25; no longer POT_D.P$2, U1.25
- net POT_R: now also IC4.23, RELEASE.P$2; no longer POT_R.P$2, U1.23
- net POT_S: now also IC4.24, SUSTAIN.P$2; no longer POT_S.P$2, U1.24
- net RST: now also IC4.29; no longer U1.29
- net SCK: now also IC3.3, IC4.17; no longer U$2.3, U1.17
- net T1: now also IC4.10, MODESW.3; no longer MODE.3, U1.10
- net T2: now also IC4.11, MODESW.1; no longer MODE.1, U1.11
- net TRIG: now also IC4.32, IC4.9, T1.3; no longer U$1.C, U1.32, U1.9
Routing:
- net +5V: track 203.9 -> 5.92 mm, vias 6 -> 0
- net 5V: track 0.00 -> 188.1 mm, vias 0 -> 6
- net N$4: track 16.7 -> 10.3 mm
- net N$7: track 14.2 -> 10.3 mm
- net +12V: track 63.6 -> 60.9 mm
- net -12V: track 74.7 -> 72.1 mm
- net N$5: track 10.8 -> 9.49 mm
- net B_TRIG: track 93.2 -> 91.9 mm
- net N$11: track 6.51 -> 5.47 mm
Other:
- board text added: "ATTACK"
- board text added: "DECAY"
- board text added: "POWER"
- board text added: "Pure ADSR V2.1"
- board text added: "RELEASE"
- board text added: "SUSTAIN"
- board text added: "T1"
- board text added: "TRIGGER BUTTON"
- board text added: "copyright GMSN Ltd 2016"
- board text removed: "Pure ADSR"

Commit message: ADSR 2.2
ADSR Updated to V2.2 14/4/21

Library updated to include 3D models.
Traces rerouted.
DAC output filter remodelled.
Power replaced so 5V comes from power supply rather than 12V, in line with low noise techniques.
Parts:
- removed C6: 47p, GMSN:C0805
- removed IC1: 78M05, GMSN:TO252
- removed POWER: HEADER2X5SHD, GMSN:2X5-SHROUDED
- removed R2: 30k, GMSN:R0805
- removed R3: 56k, GMSN:R0805
- added JP1: HEADER2X8, GMSN:POWER_SHROUDED
- C3: value 10nF -> 100nF
- MODESW: device GMSN:TOGGLE_ON_OFF_ON -> GMSN:TOGGLE_SW
- R1: value 56k -> 1k6
- moved C4 22.7 mm to (17.1, 45.1)
- moved C5 17.7 mm to (16.8, 37.9), turned to 270 degrees
- moved D1 16.3 mm to (17.1, 31.8)
- moved D2 15.4 mm to (32.4, 33.8), turned to 90 degrees
- moved C7 10.9 mm to (6.67, 51.8), turned to 0 degrees
- moved U$2 10.4 mm to (26.5, 50.8)
Connections:
- removed net +5V: C7.+, IC1.2
- removed net N$10: D2.C, POWER.1, POWER.2
- removed net N$11: C6.2, IC2.1, R8.1
- removed net N$6: OUTPUT.TIP, R2.2, R8.2
- new net N$13: D2.C, JP1.1, JP1.2
- new net N$19: D1.A, JP1.10, JP1.9
- net +12V: no longer IC1.1
- net 5V: now also C7.+, JP1.11, JP1.12
- net GND: now also JP1.3, JP1.4, JP1.5, JP1.6, JP1.7, JP1.8; no longer IC1.3, POWER.3, POWER.4, POWER.5, POWER.6, POWER.7, POWER.8, R3.1
- net N$5: now also IC2.1, R8.1; no longer C6.1, R2.1, R3.2
- net N$9: now also OUTPUT.TIP, R8.2; no longer D1.A, POWER.10, POWER.9
Routing:
- net 5V: track 188.1 -> 238.6 mm, vias 6 -> 7
- net N$6: track 42.8 -> 0.00 mm, vias 1 -> 0
- net N$13: track 0.00 -> 34.6 mm
- net N$9: track 19.0 -> 37.1 mm, vias 0 -> 1
- net +12V: track 60.9 -> 49.1 mm
- net N$10: track 9.96 -> 0.00 mm
- net -12V: track 72.1 -> 82.0 mm
- net N$19: track 0.00 -> 8.03 mm
- net +5V: track 5.92 -> 0.00 mm
- net N$4: track 10.3 -> 16.0 mm
- net N$11: track 5.47 -> 0.00 mm
- net N$5: track 9.49 -> 7.86 mm
- net RST: track 22.5 -> 24.1 mm
- net N$7: track 10.3 -> 11.5 mm
Other:
- board text added: "Pure ADSR V2.2 cc-by 4.0 2021 The Little Red Hen"
- board text removed: "POWER"
- board text removed: "Pure ADSR V2.1"
- board text removed: "copyright GMSN Ltd 2016"

Commit message: Reinstall
Parts:
- T1: value MMBT2222A -> 2N3904
Changed lines of the file:
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@@
 <drawing>
 <settings>
-<setting alwaysvectorfont="yes"/>
+<setting alwaysvectorfont="no"/>
 <setting keepoldvectorfont="yes"/>
 <setting verticaltext="up"/>
@@
 <attribute name="VALUE" x="7.62" y="65.88125" size="0.8128" layer="27" ratio="13" rot="R180"/>
 </element>
-<element name="T1" library="GMSN" library_urn="urn:adsk.eagle:library:27425118" package="SOT23" package3d_urn="urn:adsk.eagle:package:27426301/1" value="MMBT2222A" x="4.28625" y="90.4875" smashed="yes" rot="R180">
+<element name="T1" library="GMSN" library_urn="urn:adsk.eagle:library:27425118" package="SOT23" package3d_urn="urn:adsk.eagle:package:27426301/1" value="2N3904" x="4.28625" y="90.4875" smashed="yes" rot="R180">
 <attribute name="SORT" value="4" x="4.28625" y="90.4875" size="1.778" layer="27" rot="R180" display="off"/>
 </element>
 <element name="IC3" library="GMSN" library_urn="urn:adsk.eagle:library:27425118" package="SOIC8" package3d_urn="urn:adsk.eagle:package:27426231/1" value="MCP4921" x="17.145" y="86.0425" smashed="yes" rot="R180">
-<attribute name="NAME" x="18.29435" y="89.82075" size="0.8128" layer="25" ratio="13" rot="SR180"/>
+<attribute name="NAME" x="17.78" y="88.9" size="0.8128" layer="25" ratio="13" rot="SR0"/>
 <attribute name="SORT" value="4" x="17.145" y="86.0425" size="1.778" layer="27" rot="R180" display="off"/>
 <attribute name="VALUE" x="14.62405" y="87.63635" size="0.8128" layer="27" ratio="13" rot="SR0"/>
